File: Hornet.kicad_pcb (KiCad board)
At the start: 2 copper layers, 22.3 x 13 mm, 7 parts, among them J1 Conn_01x04_Female, U1 AP63203WU

Commit message: First layout
Parts:
- moved C1 0.22 mm to (126.9, 91.6)
Routing:
- net 3.3v: track 2.28 -> 0.04 mm
Changed lines of the file:
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@@
   )
   (setup
+    (stackup
+      (layer "F.SilkS" (type "Top Silk Screen"))
+      (layer "F.Paste" (type "Top Solder Paste"))
+      (layer "F.Mask" (type "Top Solder Mask") (thickness 0.01))
+      (layer "F.Cu" (type "copper") (thickness 0.035))
+      (layer "dielectric 1" (type "core") (thickness 1.51) (material "FR4") (epsilon_r 4.5) (loss_tangent 0.02))
+      (layer "B.Cu" (type "copper") (thickness 0.035))
+      (layer "B.Mask" (type "Bottom Solder Mask") (thickness 0.01))
+      (layer "B.Paste" (type "Bottom Solder Paste"))
+      (layer "B.SilkS" (type "Bottom Silk Screen"))
+      (copper_finish "None")
+      (dielectric_constraints no)
+    )
     (pad_to_mask_clearance 0)
     (pcbplotparams
@@
   )
   (footprint "Capacitor_SMD:C_0603_1608Metric" (layer "F.Cu")
-    (at 126.9746 91.7956)
+    (at 126.8984 91.5924)
     (descr "Capacitor SMD 0603 (1608 Metric), square (rectangular) end terminal, IPC_7351 nominal, (Body size source: IPC-SM-782 page 76, https://www.pcb-3d.com/wordpress/wp-content/uploads/ipc-sm-782a_amendment_1_and_2.pdf), generated with kicad-footprint-generator")
     (tags "capacitor")
@@
     )
   )
+  (gr_circle (center 115.012075 94.0308) (end 116.485275 93.98) (layer "F.Cu") (width 0.1) (fill none))
   (gr_rect (start 117.5766 83.4898) (end 139.8778 96.4438) (layer "Edge.Cuts") (width 0.1) (fill none))
   (segment (start 125.6491 89.9668) (end 125.7355 90.0532) (width 0.25) (layer "F.Cu") (net 1))
@@
   (segment (start 120.2182 91.2876) (end 122.8598 91.2876) (width 0.25) (layer "F.Cu") (net 3))
   (segment (start 125.7101 88.1278) (end 125.7355 88.1532) (width 0.25) (layer "F.Cu") (net 4))
-  (segment (start 123.4796 88.1278) (end 125.7101 88.1278) (width 0.25) (layer "F.Cu") (net 4))
-  (segment (start 123.4694 88.138) (end 123.4796 88.1278) (width 0.25) (layer "F.Cu") (net 4))
   (segment (start 126.0726 86.4362) (end 124.9172 86.4362) (width 0.25) (layer "F.Cu") (net 5))
   (segment (start 128.0105 89.1032) (end 129.3622 89.1032) (width 0.25) (layer "F.Cu") (net 5))
@@
   (segment (start 127.6226 86.4362) (end 127.6226 87.7653) (width 0.25) (layer "F.Cu") (net 6))
   (zone (net 4) (net_name "3.3v") (layer "F.Cu") (hatch edge 0.508)
-    (connect_pads thru_hole_only (clearance 0.254))
+    (connect_pads yes (clearance 0.254))
     (min_thickness 0.254) (filled_areas_thickness no)
-    (fill yes (thermal_gap 0.508) (thermal_bridge_width 0.508))
+    (fill yes (thermal_gap 0.508) (thermal_bridge_width 0.508) (smoothing fillet) (radius 0.5))
     (polygon
       (pts
-        (xy 117.7544 90.17)
-        (xy 117.729 87.122)
-        (xy 117.7544 83.6676)
-        (xy 121.332232 83.486677)
+        (xy 121.665212 88.743731)
+        (xy 121.645351 88.502151)
+        (xy 121.586299 88.267059)
+        (xy 121.489645 88.044768)
+        (xy 121.357982 87.841248)
+        (xy 121.194847 87.661965)
+        (xy 121.004621 87.511734)
+        (xy 120.792413 87.394589)
+        (xy 120.563921 87.313675)
+        (xy 120.325282 87.271167)
+        (xy 120.082905 87.268206)
+        (xy 119.843299 87.304871)
+        (xy 119.612899 87.380177)
+        (xy 119.397892 87.492103)
+        (xy 119.204052 87.637642)
+        (xy 119.036586 87.812886)
+        (xy 118.89999 88.013128)
+        (xy 118.797933 88.232991)
+        (xy 118.733155 88.46657)
+        (xy 118.707398 88.707593)
+        (xy 118.721351 88.949586)
+        (xy 118.77464 89.186051)
+        (xy 118.865835 89.410637)
+        (xy 118.992486 89.617312)
+        (xy 119.151192 89.800528)
+        (xy 119.337691 89.955362)
+        (xy 119.546974 90.077657)
+        (xy 119.77342 90.164128)
+        (xy 120.010949 90.212454)
+        (xy 120.253182 90.221336)
+        (xy 120.493612 90.190537)
+        (xy 120.725783 90.120882)
+        (xy 120.943461 90.014243)
+        (xy 121.140799 89.873483)
+        (xy 121.312497 89.702383)
+        (xy 121.453944 89.505538)
+        (xy 121.561342 89.288234)
+        (xy 121.631807 89.056307)
+        (xy 121.663446 88.815986)
+      )
+    )
+  )
+  (zone (net 4) (net_name "3.3v") (layer "F.Cu") (hatch edge 0.508)
+    (connect_pads yes (clearance 0.254))
+    (min_thickness 0.254) (filled_areas_thickness no)
+    (fill yes (thermal_gap 0.508) (thermal_bridge_width 0.508) (smoothing fillet) (radius 0.5))
+    (polygon
+      (pts
+        (xy 119.888 90.17)
+        (xy 119.888 87.3252)
+        (xy 122.0216 87.3252)
+        (xy 122.0216 83.5152)
         (xy 137.6172 83.4898)
         (xy 137.6934 91.5162)
         (xy 135.4836 95.2754)
         (xy 133.604 95.2754)
-        (xy 133.6802 84.8106)
-        (xy 129.0066 84.836)
-        (xy 124.322917 85.2678)
+        (xy 133.681856 85.115389)
+        (xy 129.008256 85.140789)
+        (xy 124.1552 85.1408)
+        (xy 124.1552 87.5792)
+        (xy 126.6444 87.63)
+        (xy 126.5936 88.5952)
         (xy 124.37377 88.566835)
-        (xy 122.8598 90.0938)
-        (xy 120.723923 90.146526)
+        (xy 122.8344 90.17)
+      )
+    )
+  )
+  (zone (net 1) (net_name "Vin") (layer "F.Cu") (hatch edge 0.508)
+    (connect_pads yes (clearance 0.254))
+    (min_thickness 0.254) (filled_areas_thickness no)
+    (fill yes (thermal_gap 0.508) (thermal_bridge_width 0.508) (smoothing fillet) (radius 0.5))
+    (polygon
+      (pts
+        (xy 126.8984 92.3544)
+        (xy 125.1204 92.3544)
+        (xy 122.2756 95.3008)
+        (xy 119.7356 95.3516)
+        (xy 119.734669 92.410401)
+        (xy 122.268849 92.405329)
+        (xy 125.1204 89.662)
+        (xy 126.8984 89.662)
       )
     )
@@
   )
   (zone (net 1) (net_name "Vin") (layer "F.Cu") (hatch edge 0.508)
-    (connect_pads thru_hole_only (clearance 0.254))
+    (connect_pads yes (clearance 0.254))
     (min_thickness 0.254) (filled_areas_thickness no)
-    (fill yes (thermal_gap 0.508) (thermal_bridge_width 0.508))
+    (fill yes (thermal_gap 0.508) (thermal_bridge_width 0.508) (smoothing fillet) (radius 0.5))
     (polygon
       (pts
-        (xy 126.8476 91.567)
-        (xy 126.91104 92.646489)
-        (xy 122.078837 96.095196)
-        (xy 118.103797 95.979589)
-        (xy 118.0592 92.202)
-        (xy 122.428 92.202)
-        (xy 125.0442 89.6366)
-        (xy 126.6698 89.6112)
+        (xy 121.671928 93.8784)
+        (xy 121.652067 93.63682)
+        (xy 121.593015 93.401728)
+        (xy 121.496361 93.179437)
+        (xy 121.364698 92.975917)
+        (xy 121.201563 92.796634)
+        (xy 121.011337 92.646403)
+        (xy 120.799129 92.529258)
+        (xy 120.570637 92.448344)
+        (xy 120.331998 92.405836)
+        (xy 120.089621 92.402875)
+        (xy 119.850015 92.43954)
+        (xy 119.619615 92.514846)
+        (xy 119.404608 92.626772)
+        (xy 119.210768 92.772311)
+        (xy 119.043302 92.947555)
+        (xy 118.906706 93.147797)
+        (xy 118.804649 93.36766)
+        (xy 118.739871 93.601239)
+        (xy 118.714114 93.842262)
+        (xy 118.728067 94.084255)
+        (xy 118.781356 94.32072)
+        (xy 118.872551 94.545306)
+        (xy 118.999202 94.751981)
+        (xy 119.157908 94.935197)
+        (xy 119.344407 95.090031)
+        (xy 119.55369 95.212326)
+        (xy 119.780136 95.298797)
+        (xy 120.017665 95.347123)
+        (xy 120.259898 95.356005)
+        (xy 120.500328 95.325206)
+        (xy 120.732499 95.255551)
+        (xy 120.950177 95.148912)
+        (xy 121.147515 95.008152)
+        (xy 121.319213 94.837052)
+        (xy 121.46066 94.640207)
+        (xy 121.568058 94.422903)
+        (xy 121.638523 94.190976)
+        (xy 121.670162 93.950655)
       )
     )
